File: hardware/compta-birres-sch/display.kicad_sch (KiCad schematic)
At the start: 5 parts, among them U2 74HC595, U3 74HC595, U4 74HC595, U5 74HC595, U6 74HC595

Commit message: Finalized buttons schematic, added tlp521-4
Parts:
- renumbered U2 to U5, U3 to U6, U4 to U7, U5 to U8, U6 to U9
Other:
- sheet Custom 7 Segment Display 1 ports: added GND; removed none
- sheet Custom 7 Segment Display 2 ports: added GND; removed none
- sheet Custom 7 Segment Display 3 ports: added GND; removed none
- sheet Custom 7 Segment Display 4 ports: added GND; removed none
- sheet Custom 7 Segment Display 5 ports: added GND; removed none
