File: hardware/compta-birres-sch/buttons.kicad_sch (KiCad schematic)
At the start: 25 parts, among them SW1 SW_Push, SW2 SW_Push, SW3 SW_Push, SW4 SW_Push, SW5 SW_Push, SW6 SW_Push, SW7 SW_Push, SW8 SW_Push, U7 74HC4051

Commit message: Finalized buttons schematic, added tlp521-4
Parts:
- removed C1, C2, C3, C4, C5, C6, C7, C8: 0.1u, symbol Device:C_45deg
- removed R1, R2, R4, R6, R8: 1k, symbol Device:R_45deg
- removed SW1: SW_Push, symbol Switch:SW_Push
- added R10, R12, R14, R16, R18, R4, R6, R8: 560, symbol Device:R
- added R11, R13, R15, R17, R9: 10k, symbol Device:R_45deg
- added SW9: SW_Push, symbol Switch:SW_Push
- added U2, U4: TLP521-4, symbol cb_lib:TLP521-4
- R3, R5, R7: value 1k -> 10k
- renumbered U7 to U3
Connections:
- net 3V3: now also R11.1, R13.1, R15.1, R17.1, R9.1
- net GND: now also U2.11 (R), U2.13 (R), U2.15 (R), U2.2 (K), U2.4 (K), U2.6 (K), U2.8 (K), U2.9 (R), U4.11 (R), U4.13 (R), U4.15 (R), U4.2 (K), U4.4 (K), U4.6 (K), U4.8 (K), U4.9 (R); no longer SW2.2, SW3.2, SW4.2, SW5.2, SW6.2, SW7.2, SW8.2
- net at U3.13 (A0): now also R3.2, U2.16 (R)
- net at U3.12 (A3): now also R9.2, U2.10 (R); no longer SW4.1
- net at U3.14 (A1): now also R5.2, U2.14 (R); no longer SW2.1
- net at U3.5 (A5): now also R13.2, U4.14 (R); no longer SW6.1
- net at U3.4 (A7): now also R17.2, U4.10 (R); no longer SW8.1
- new net: R15.2, U3.2 (A6), U4.12 (R)
- new net: R8.2, SW4.2
- new net: R11.2, U3.1 (A4), U4.16 (R)
- new net: R6.1, U2.3 (A)
- new net: R16.1, U4.5 (A)
- new net: R12.1, U4.1 (A)
- new net: R6.2, SW3.2
- new net: R18.1, U4.7 (A)
- new net: R18.2, SW9.2
- new net: R10.1, U2.7 (A)
- new net: R10.2, SW5.2
- new net: R8.1, U2.5 (A)
- new net: R16.2, SW8.2
- new net: R14.1, U4.3 (A)
- new net: R14.2, SW7.2
- new net: R7.2, U2.12 (R), U3.15 (A2)
- new net: R12.2, SW6.2
- new net: R4.2, SW2.2
- new net: R4.1, U2.1 (A)
- new net 12V: SW2.1, SW3.1, SW4.1, SW5.1, SW6.1, SW7.1, SW8.1, SW9.1

Commit message: Annotated schematic
Changed lines of the file:
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@@
 	(title_block
 		(title "Buttons")
-		(date "2024-09-24")
-		(rev "1.2")
+		(date "2024-09-26")
+		(rev "1.3")
 		(company "Associació Cultural TGK")
 		(comment 1 "Author: lluc")
@@
 		)
 	)
+	(text_box "Ra (Anode resistor on optocoupler) Calculation:\n\nVf = 1.15 V\nif = 20 mA\n\nRa = (Vcc - Vf)/If = 542 Ohms -> 560 Ohms\n\nP = Ra * If^2 = 0.35 W -> 1/2 W"
+		(exclude_from_sim no)
+		(at 17.78 17.78 0)
+		(size 50.8 17.78)
+		(stroke
+			(width 0)
+			(type default)
+		)
+		(fill
+			(type color)
+			(color 255 229 191 1)
+		)
+		(effects
+			(font
+				(size 1.27 1.27)
+			)
+			(justify left top)
+		)
+	)
