File: hardware/compta-birres-sch/cstm_7seg.kicad_sch (KiCad schematic)
At the start: 46 parts, among them Q17 2N7000, Q18 2N7000, Q19 2N7000, Q20 2N7000, Q21 2N7000, Q22 2N7000, Q23 2N7000, Q24 2N7000

Commit message: Finalized buttons schematic, added tlp521-4
Parts:
- removed AFF2: LTS-6960HR, Display_7Segment:7SegmentLED_LTS6760_LTS6780, symbol Display_Character:LTS-6960HR
- added AFF2: LTS-6980HR, Display_7Segment:7SegmentLED_LTS6760_LTS6780, symbol Display_Character:LTS-6980HR
- renumbered D49 to D1, D50 to D10, D53 to D11, D56 to D12, D46 to D13, D61 to D14, D47 to D15, D62 to D16, D48 to D17, D63 to D18, D51 to D19, D52 to D2, D54 to D20, D57 to D21, D55 to D3, D43 to D4, D58 to D5, D44 to D6, D59 to D7, D45 to D8, D60 to D9, Q17 to Q1, Q21 to Q2, Q18 to Q3, Q22 to Q4, Q19 to Q5, Q23 to Q6, Q20 to Q7, Q24 to Q8, R43 to R19, R51 to R20, R47 to R21, R55 to R22, R44 to R23, R52 to R24, R48 to R25, R56 to R26, R45 to R27, R53 to R28, R49 to R29, R57 to R30, R46 to R31, R54 to R32, R50 to R33, R58 to R34
Connections:
- net GND: now also Q8.1 (S), R34.2, AFF2.3 (C.K.), AFF2.8 (C.K.)
- net a: now also AFF2.7 (a)
- net b: now also AFF2.6 (b)
- net c: now also AFF2.4 (c)
- net d: now also AFF2.2 (d)
- net dp: now also AFF2.5 (DP)
- net e: now also AFF2.1 (e)
- net f: now also AFF2.9 (f)
- net g: now also AFF2.10 (g)

Commit message: Annotated schematic
Parts:
- renumbered AFF2 to AFF3, D1 to D43, D2 to D44, D3 to D45, D4 to D46, D5 to D47, D6 to D48, D7 to D49, D8 to D50, D9 to D51, D10 to D52, D11 to D53, D12 to D54, D13 to D55, D14 to D56, D15 to D57, D16 to D58, D17 to D59, D18 to D60, D19 to D61, D20 to D62, D21 to D63, Q1 to Q17, Q2 to Q18, Q3 to Q19, Q4 to Q20, Q5 to Q21, Q6 to Q22, Q7 to Q23, Q8 to Q24, R19 to R51, R20 to R52, R21 to R53, R22 to R54, R23 to R55, R24 to R56, R25 to R57, R26 to R58, R27 to R59, R28 to R60, R29 to R61, R30 to R62, R31 to R63, R32 to R64, R33 to R65, R34 to R66
Changed lines of the file:
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@@
 		(dnp no)
 		(fields_autoplaced yes)
-		(property "Reference" "D16"
+		(property "Reference" "D58"
 			(at 97.79 144.4625 0)
 			(effects
@@
 		(dnp no)
 		(fields_autoplaced yes)
-		(property "Reference" "R21"
+		(property "Reference" "R53"
 			(at 167.64 38.0999 0)
 			(effects
@@
 		(dnp no)
 		(fields_autoplaced yes)
-		(property "Reference" "R19"
+		(property "Reference" "R51"
 			(at 156.21 25.4 90)
 			(effects
@@
 		(dnp no)
 		(fields_autoplaced yes)
-		(property "Reference" "Q8"
+		(property "Reference" "Q24"
 			(at 245.11 125.7299 0)
 			(effects
@@
 		(dnp no)
 		(fields_autoplaced yes)
-		(property "Reference" "D5"
+		(property "Reference" "D47"
 			(at 97.79 50.4825 0)
 			(effects
@@
 		(dnp no)
 		(fields_autoplaced yes)
-		(property "Reference" "Q5"
+		(property "Reference" "Q21"
 			(at 181.61 93.9799 0)
 			(effects
@@
 		(dnp no)
 		(fields_autoplaced yes)
-		(property "Reference" "Q2"
+		(property "Reference" "Q18"
 			(at 245.11 30.4799 0)
 			(effects
@@
 		(dnp no)
 		(fields_autoplaced yes)
-		(property "Reference" "D18"
+		(property "Reference" "D60"
 			(at 97.79 157.1625 0)
 			(effects
@@
 		(dnp no)
 		(fields_autoplaced yes)
-		(property "Reference" "D11"
+		(property "Reference" "D53"
 			(at 66.3575 97.79 0)
 			(effects
@@
 		(dnp no)
 		(fields_autoplaced yes)
-		(property "Reference" "R22"
+		(property "Reference" "R54"
 			(at 231.14 38.0999 0)
 			(effects
@@
 		(dnp no)
 		(fields_autoplaced yes)
-		(property "Reference" "R32"
+		(property "Reference" "R64"
 			(at 219.71 120.65 90)
 			(effects
@@
 		(dnp no)
 		(fields_autoplaced yes)
-		(property "Reference" "D6"
+		(property "Reference" "D48"
 			(at 29.21 75.8825 0)
 			(effects
@@
 		(dnp no)
 		(fields_autoplaced yes)
-		(property "Reference" "Q3"
+		(property "Reference" "Q19"
 			(at 181.61 62.2299 0)
 			(effects
@@
 		(dnp no)
 		(fields_autoplaced yes)
-		(property "Reference" "D12"
+		(property "Reference" "D54"
 			(at 91.7575 97.79 0)
 			(effects
@@
 		(dnp no)
 		(fields_autoplaced yes)
-		(property "Reference" "R20"
+		(property "Reference" "R52"
 			(at 219.71 25.4 90)
 			(effects
@@
 		(dnp no)
 		(fields_autoplaced yes)
-		(property "Reference" "R27"
+		(property "Reference" "R59"
 			(at 156.21 88.9 90)
 			(effects
@@
 		(dnp no)
 		(fields_autoplaced yes)
-		(property "Reference" "R25"
+		(property "Reference" "R57"
 			(at 167.64 69.8499 0)
 			(effects
@@
 		(dnp no)
 		(fields_autoplaced yes)
-		(property "Reference" "R28"
+		(property "Reference" "R60"
 			(at 219.71 88.9 90)
 			(effects
@@
 		(dnp no)
 		(fields_autoplaced yes)
-		(property "Reference" "AFF2"
+		(property "Reference" "AFF3"
 			(at 147.32 160.02 0)
 			(effects
@@
 		(dnp no)
 		(fields_autoplaced yes)
-		(property "Reference" "D4"
+		(property "Reference" "D46"
 			(at 29.21 50.4825 0)
 			(effects
@@
 		(dnp no)
 		(fields_autoplaced yes)
-		(property "Reference" "D19"
+		(property "Reference" "D61"
 			(at 53.6575 166.37 0)
 			(effects
@@
 		(dnp no)
 		(fields_autoplaced yes)
-		(property "Reference" "D2"
+		(property "Reference" "D44"
 			(at 66.3575 29.21 0)
 			(effects
@@
 		(dnp no)
 		(fields_autoplaced yes)
-		(property "Reference" "R24"
+		(property "Reference" "R56"
 			(at 219.71 57.15 90)
 			(effects
@@
 		(dnp no)
 		(fields_autoplaced yes)
-		(property "Reference" "D14"
+		(property "Reference" "D56"
 			(at 97.79 119.0625 0)
 			(effects
@@
 		(dnp no)
 		(fields_autoplaced yes)
-		(property "Reference" "R31"
+		(property "Reference" "R63"
 			(at 156.21 120.65 90)
 			(effects
@@
 		(dnp no)
 		(fields_autoplaced yes)
-		(property "Reference" "D9"
+		(property "Reference" "D51"
 			(at 97.79 88.5825 0)
 			(effects
@@
 		(dnp no)
 		(fields_autoplaced yes)
-		(property "Reference" "Q4"
+		(property "Reference" "Q20"
 			(at 245.11 62.2299 0)
 			(effects
@@
 		(dnp no)
 		(fields_autoplaced yes)
-		(property "Reference" "D3"
+		(property "Reference" "D45"
 			(at 91.7575 29.21 0)
 			(effects
@@
 		(dnp no)
 		(fields_autoplaced yes)
-		(property "Reference" "R29"
+		(property "Reference" "R61"
 			(at 167.64 101.5999 0)
 			(effects
@@
 		(dnp no)
 		(fields_autoplaced yes)
-		(property "Reference" "R34"
+		(property "Reference" "R66"
 			(at 231.14 133.3499 0)
 			(effects
@@
 		(dnp no)
 		(fields_autoplaced yes)
-		(property "Reference" "D13"
+		(property "Reference" "D55"
 			(at 29.21 119.0625 0)
 			(effects
@@
 		(dnp no)
 		(fields_autoplaced yes)
-		(property "Reference" "Q7"
+		(property "Reference" "Q23"
 			(at 181.61 125.7299 0)
 			(effects
@@
 		(dnp no)
 		(fields_autoplaced yes)
-		(property "Reference" "D15"
+		(property "Reference" "D57"
 			(at 29.21 144.4625 0)
 			(effects
@@
 		(dnp no)
 		(fields_autoplaced yes)
-		(property "Reference" "D21"
+		(property "Reference" "D63"
 			(at 91.7575 166.37 0)
 			(effects
@@
 		(dnp no)
 		(fields_autoplaced yes)
-		(property "Reference" "R33"
+		(property "Reference" "R65"
 			(at 167.64 133.3499 0)
 			(effects
@@
 		(dnp no)
 		(fields_autoplaced yes)
-		(property "Reference" "R30"
+		(property "Reference" "R62"
 			(at 231.14 101.5999 0)
 			(effects
@@
 		(dnp no)
 		(fields_autoplaced yes)
-		(property "Reference" "Q6"
+		(property "Reference" "Q22"
 			(at 245.11 93.9799 0)
 			(effects
@@
 		(dnp no)
 		(fields_autoplaced yes)
-		(property "Reference" "D1"
+		(property "Reference" "D43"
 			(at 53.6575 29.21 0)
 			(effects
@@
 		(dnp no)
 		(fields_autoplaced yes)
-		(property "Reference" "D20"
+		(property "Reference" "D62"
 			(at 66.3575 166.37 0)
 			(effects
@@
 		(dnp no)
 		(fields_autoplaced yes)
-		(property "Reference" "D10"
+		(property "Reference" "D52"
 			(at 53.6575 97.79 0)
 			(effects
@@
 		(dnp no)
 		(fields_autoplaced yes)
-		(property "Reference" "R26"
+		(property "Reference" "R58"
 			(at 231.14 69.8499 0)
 			(effects
@@
 		(dnp no)
 		(fields_autoplaced yes)
-		(property "Reference" "D7"
+		(property "Reference" "D49"
 			(at 97.79 75.8825 0)
 			(effects
@@
 		(dnp no)
 		(fields_autoplaced yes)
-		(property "Reference" "R23"
+		(property "Reference" "R55"
 			(at 156.21 57.15 90)
 			(effects
@@
 		(dnp no)
 		(fields_autoplaced yes)
-		(property "Reference" "Q1"
+		(property "Reference" "Q17"
 			(at 181.61 30.4799 0)
 			(effects
@@
 		(dnp no)
 		(fields_autoplaced yes)
-		(property "Reference" "D8"
+		(property "Reference" "D50"
 			(at 29.21 88.5825 0)
 			(effects
@@
 		(dnp no)
 		(fields_autoplaced yes)
-		(property "Reference" "D17"
+		(property "Reference" "D59"
 			(at 29.21 157.1625 0)
 			(effects
